Commit message: fix: wheel position and controller  manager

File: ros_ws/src/simple_robot_description/models/robot/robot.gazebo.xacro (robot description, xacro)
@@ -42,6 +42,6 @@
 <gazebo>
     <plugin name="gazebo_ros2_control" filename="libgazebo_ros2_control.so">
-        <robot_sim_type>gazebo_ros2_control/DefaultRobotHWSim</robot_sim_type>
-        <!-- <robot_sim_type>gazebo_ros2_control/GazeboSystem</robot_sim_type> -->
+        <!-- <robot_sim_type>gazebo_ros2_control/DefaultRobotHWSim</robot_sim_type> -->
+        <robot_sim_type>gazebo_ros2_control/GazeboSystem</robot_sim_type>
         <parameters>/home/a/robotics-lab/final-project/robotics-assignment/ros_ws/src/simple_robot_description/config/robot.yaml</parameters>
     </plugin>

File: ros_ws/src/simple_robot_description/models/robot/robot.urdf (robot description, URDF)
Before this commit: robot four_wheel_robot, 6 links, 5 joints
Links:
- link wheel1_link: mass -19.155861183375002 -> 19.155861183375002
- link wheel2_link: mass -19.155861183375002 -> 19.155861183375002
- link wheel3_link: mass -19.155861183375002 -> 19.155861183375002
- link wheel4_link: mass -19.155861183375002 -> 19.155861183375002

File: ros_ws/src/simple_robot_description/models/robot/robot.xacro (robot description, xacro)
@@ -1,4 +1,4 @@
 <?xml version="1.0"?>
-<robot name="four_wheel_robot" xmlns:xacro="http://www.ros.org/wiki/xacro">
+<robot name="robot" xmlns:xacro="http://www.ros.org/wiki/xacro">
 <!-- Body -->
 <xacro:property name="body_link_x_dim" value="1" />
@@ -16,5 +16,5 @@
 <!-- Robod body and wheel mass -->
 <xacro:property name="body_mass" value="${body_density*body_link_x_dim*body_link_y_dim*body_link_z_dim}" />
-<xacro:property name="wheel_mass" value="${-wheel_density*pi_const*wheel_link_radius*wheel_link_radius*wheel_link_length}" />
+<xacro:property name="wheel_mass" value="${wheel_density*pi_const*wheel_link_radius*wheel_link_radius*wheel_link_length}" />
 <!-- Moment of inertia of the whee -->
 <xacro:property name="Iz_wheel" value="${0.5*wheel_mass*wheel_link_radius*wheel_link_radius}" />

Commit message: feat: keyboard controlled 4wr

File: ros_ws/src/simple_robot_description/models/robot/robot.gazebo.xacro (robot description, xacro)
@@ -2,26 +2,36 @@
 <robot>
 <gazebo reference="body_link">
-<mu1>0.2</mu1>
-<mu2>0.2</mu2>
+<kp>1000000.0</kp>
+<kd>100.0</kd>
+<mu1>1.0</mu1>
+<mu2>1.0</mu2>
 <material>Gazebo/Red</material>
 </gazebo>
 <gazebo reference="wheel1_link">
-<mu1>0.2</mu1>
-<mu2>0.2</mu2>
+<kp>1000000.0</kp>
+<kd>100.0</kd>
+<mu1>1.0</mu1>
+<mu2>1.0</mu2>
 <material>Gazebo/Yellow</material>
 </gazebo>
 <gazebo reference="wheel2_link">
-<mu1>0.2</mu1>
-<mu2>0.2</mu2>
+<kp>1000000.0</kp>
+<kd>100.0</kd>
+<mu1>1.0</mu1>
+<mu2>1.0</mu2>
 <material>Gazebo/Yellow</material>
 </gazebo>
 <gazebo reference="wheel3_link">
-<mu1>0.2</mu1>
-<mu2>0.2</mu2>
+<kp>1000000.0</kp>
+<kd>100.0</kd>
+<mu1>1.0</mu1>
+<mu2>1.0</mu2>
 <material>Gazebo/Yellow</material>
 </gazebo>
 <gazebo reference="wheel4_link">
-<mu1>0.2</mu1>
-<mu2>0.2</mu2>
+<kp>1000000.0</kp>
+<kd>100.0</kd>
+<mu1>1.0</mu1>
+<mu2>1.0</mu2>
 <material>Gazebo/Yellow</material>
 </gazebo>
@@ -30,5 +40,5 @@
         <plugin>gazebo_ros2_control/GazeboSystem</plugin>
     </hardware>
-    <joint name="joint1">
+    <!-- <joint name="wheel1_joint">
         <command_interface name="position">
             <param name="min">-6.2832</param>
@@ -38,5 +48,5 @@
         <state_interface name="velocity" />
         <state_interface name="effort" />
-    </joint>
+    </joint> -->
 </ros2_control>
 <gazebo>
@@ -47,3 +57,28 @@
     </plugin>
 </gazebo>
+<gazebo>
+    <plugin name="skid_steer_drive_controller" filename="libgazebo_ros_diff_drive.so">
+        <update_rate>500</update_rate>
+        <num_wheel_pairs>2</num_wheel_pairs>
+        <left_joint>wheel2_joint</left_joint>
+        <right_joint>wheel1_joint</right_joint>
+        <left_joint>wheel4_joint</left_joint>
+        <right_joint>wheel3_joint</right_joint>
+        <wheel_separation>${body_link_y_dim+wheel_link_length}</wheel_separation>
+        <wheel_separation>${body_link_y_dim+wheel_link_length}</wheel_separation>
+        <wheel_diameter>${2*wheel_link_radius}</wheel_diameter>
+        <wheel_diameter>${2*wheel_link_radius}</wheel_diameter>
+        <max_wheel_torque>200</max_wheel_torque>
+        <max_wheel_acceleration>10.0</max_wheel_acceleration>
+        <command_topic>cmd_vel</command_topic>
+        <odometry_topic>odom</odometry_topic>
+        <odometry_frame>odom</odometry_frame>
+        <robot_base_frame>dummy</robot_base_frame>
+        <publish_wheel_tf>true</publish_wheel_tf>
+        <publish_odom>true</publish_odom>
+        <covariance_x>0.0001</covariance_x>
+        <covariance_y>0.0001</covariance_y>
+        <covariance_yaw>0.01</covariance_yaw>
+    </plugin>
+</gazebo>
 </robot>

File: ros_ws/src/simple_robot_description/models/robot/robot.xacro (robot description, xacro)
@@ -40,5 +40,5 @@
             <box size="${body_link_x_dim} ${body_link_y_dim} ${body_link_z_dim}" />
         </geometry>
-        <origin rpy="0 0 0" xyz="0 0 0" />
+        <origin rpy="0 0 0" xyz="0 0 0.25" />
     </visual>
     <collision>
@@ -46,8 +46,8 @@
             <box size="${body_link_x_dim} ${body_link_y_dim} ${body_link_z_dim}" />
         </geometry>
-        <origin rpy="0 0 0" xyz="0 0 0" />
+        <origin rpy="0 0 0" xyz="0 0 0.25" />
     </collision>
     <inertial>
-        <origin rpy="0 0 0" xyz="0 0 0" />
+        <origin rpy="0 0 0" xyz="0 0 0.25" />
         <mass value="${body_mass}" />
         <inertia
